Commit message: changed type of tool joint from "revolute" to "continuous"

File: pantograph_description/urdf/pantograph.urdf.xacro (robot description, xacro)
@@ -159,9 +159,8 @@
   <!-- tool pitch angle-->
   <link name="tool_theta_link"/>
-  <joint name="tool_theta_joint" type="revolute">
+  <joint name="tool_theta_joint" type="continuous">
     <parent link= "panto_tool0"/>
     <child link= "tool_theta_link"/>
     <origin xyz = "0 0 0" rpy="0 0 0"/>
-    <limit effort="1000.0" lower="-3" upper="3" velocity="0.5"/>
     <axis xyz="0 0 1"/>
   </joint>
@@ -176,9 +175,8 @@
     </visual>
   </link>
-  <joint name="tool_phi_joint" type="revolute">
+  <joint name="tool_phi_joint" type="continuous">
     <origin rpy="0 0 0" xyz="0 0 0"/>
     <parent link="tool_theta_link"/>
     <child link="tool_phi_link"/>
-    <limit effort="1000.0" lower="-3" upper="3" velocity="0.5"/>
     <axis xyz="0 1 0"/>
   </joint>
