Commit message: add meshes + fix joints

File: pantograph_description/ros2_control/pantograph.r2c_hardware.xacro (robot description, xacro)
@@ -24,5 +24,5 @@
       </xacro:unless>
       <!-- Actual joints (i.e., motors) -->
-      <joint name="panto_left_joint">
+      <joint name="panto_a1">
         <command_interface name="${command_interface}" />
         <state_interface name="force">
@@ -32,5 +32,5 @@
         </state_interface>
         <state_interface name="position">
-          <param name="initial_value">0.7498</param>
+          <param name="initial_value">${1.57 + 0.5}</param>
           <param name="min">-1.57</param>
           <param name="max">1.57</param>
@@ -45,10 +45,10 @@
               <param name="alias"> 0 </param>
               <param name="position"> 2 </param>
-              <param name="slave_config">$(find ${ec_config_package})/config/beckhoff_el5101.yaml</param>
+              <param name="slave_config">$(find ${ec_config_package})/config/beckhoff_el5101_left.yaml</param>
             </ec_module>
           </xacro:unless>
         </xacro:unless>
       </joint>
-      <joint name="panto_right_joint">
+      <joint name="panto_a5">
           <command_interface name="${command_interface}"/>
           <state_interface name="force">
@@ -58,5 +58,5 @@
           </state_interface>
           <state_interface name="position">
-              <param name="initial_value">0.7498</param>
+              <param name="initial_value">0.5</param>
               <param name="min">-1.57</param>
               <param name="max">1.57</param>
@@ -71,5 +71,5 @@
                 <param name="alias"> 0 </param>
                 <param name="position"> 1 </param>
-                <param name="slave_config">$(find ${ec_config_package})/config/beckhoff_el5101.yaml</param>
+                <param name="slave_config">$(find ${ec_config_package})/config/beckhoff_el5101_right.yaml</param>
               </ec_module>
             </xacro:unless>
@@ -77,4 +77,37 @@
       </joint>
       <!-- Mock joints used for visualization -->
+      <joint name="panto_a2">
+          <command_interface name="position"/>
+          <state_interface name="position">
+              <param name="initial_value">${-1.4}</param>
+              <param name="min">-1.57</param>
+              <param name="max">1.57</param>
+          </state_interface>
+          <state_interface name="velocity">
+              <param name="initial_value">0.0</param>
+          </state_interface>
+      </joint>
+      <joint name="panto_a3">
+          <command_interface name="position"/>
+          <state_interface name="position">
+              <param name="initial_value">${- 1.57 - 0.5 + 1.4}</param>
+              <param name="min">-1.57</param>
+              <param name="max">1.57</param>
+          </state_interface>
+          <state_interface name="velocity">
+              <param name="initial_value">0.0</param>
+          </state_interface>
+      </joint>
+      <joint name="panto_a4">
+          <command_interface name="position"/>
+          <state_interface name="position">
+              <param name="initial_value">${1.65}</param>
+              <param name="min">-1.57</param>
+              <param name="max">1.57</param>
+          </state_interface>
+          <state_interface name="velocity">
+              <param name="initial_value">0.0</param>
+          </state_interface>
+      </joint>
     </ros2_control>
   </xacro:macro>

File: pantograph_description/urdf/pantograph.urdf.xacro (robot description, xacro)
@@ -2,4 +2,7 @@
 <robot xmlns:xacro="http://www.ros.org/wiki/xacro">
   <xacro:macro name="pantograph" params="parent *origin">
+  <material name="white_alpha">
+    <color rgba="${255/255} ${255/255} ${255/255} 0.6"/>
+  </material>
   <material name="blue">
     <color rgba="0.0 0.0 0.8 1.0"/>
@@ -15,7 +18,7 @@
     <visual>
       <geometry>
-        <box size = "0.082 0.050 0.03"/>
+        <mesh filename="package://pantograph_description/meshes/mesh_base.stl" scale="0.001 0.001 0.001"/>
       </geometry>
-      <material name = "blue"/>
+      <material name = "white_alpha"/>
       <origin xyz="0 0 0" rpy="0 0 0" />
     </visual>
@@ -26,18 +29,96 @@
       <child link="panto_base"/>
   </joint>
+  <!-- ==========  Fulcrum =========== -->
+  <link name = "panto_link_fulcrum">
+    <visual>
+      <geometry>
+        <mesh filename="package://pantograph_description/meshes/mesh_fulcrum.stl" scale="0.001 0.001 0.001"/>
+      </geometry>
+      <material name = "white_alpha"/>
+      <origin xyz = "0 0 0" rpy = "0 0 0"/>
+    </visual>
+  </link>
+  <joint name = "panto_base_to_fulcrum" type="fixed">
+    <parent link = "panto_base"/>
+    <child link = "panto_link_fulcrum"/>
+    <origin xyz = "0.0425 0.16056 0.09"/>
+  </joint>
+  <!-- ==========  Left arm (as seen from behind) =========== -->
+  <link name = "panto_left_motor">
+    <inertial>
+      <!-- izz = 69.9 g/cm², see https://www.farnell.com/datasheets/484832.pdf -->
+      <mass value="0.1"/>
+      <inertia ixx="0.1" ixy="0.0" ixz="0.0" iyy="0.1" iyz="0.0" izz="0.00000699"/>
+    </inertial>
+  </link>
+  <joint name = "panto_a1" type="revolute">
+    <parent link = "panto_base"/>
+    <child link = "panto_left_motor"/>
+    <origin xyz = "0.0 0 0" rpy="0 0 0"/>
+    <limit effort="1000.0" lower="-1.57" upper="1.57" velocity="0.5"/>
+    <axis xyz = "0 0 1"/>
+    <dynamics damping="0.2" friction="0.1" />
+  </joint>
+  <link name = "panto_left_link1">
+    <visual>
+      <geometry>
+        <mesh filename="package://pantograph_description/meshes/mesh_link_left_1.stl" scale="0.001 0.001 0.001"/>
+      </geometry>
+      <material name = "green"/>
+      <origin xyz = "0 0 0" rpy = "0 0 0"/>
+    </visual>
+  </link>
+  <joint name = "panto_left_motor_to_link1" type="fixed">
+    <parent link = "panto_left_motor"/>
+    <child link = "panto_left_link1"/>
+    <origin xyz = "0 0 0"/>
+  </joint>
+  <link name = "panto_left_link2">
+    <visual>
+      <geometry>
+        <mesh filename="package://pantograph_description/meshes/mesh_link_left_2.stl" scale="0.001 0.001 0.001"/>
+      </geometry>
+      <material name = "green"/>
+      <origin xyz = "0 0 0" rpy = "0 0 0"/>
+    </visual>
+  </link>
+  <joint name = "panto_a2" type="revolute">
+    <parent link = "panto_left_link1"/>
+    <child link = "panto_left_link2"/>
+    <origin xyz = "0.1 0 0" rpy="0 0 0"/>
+    <limit effort="1000.0" lower="-1.57" upper="1.57" velocity="0.5"/>
+    <axis xyz = "0 0 1"/>
+    <dynamics damping="0.2" friction="0.1" />
+  </joint>
+  <!-- ==========  Tool link (orange sphere) =========== -->
+  <link name = "panto_tool0">
+    <visual>
+      <geometry>
+        <mesh filename="package://pantograph_description/meshes/mesh_tool0.stl" scale="0.001 0.001 0.001"/>
+      </geometry>
+      <material name = "orange"/>
+      <origin xyz = "0 0 0" rpy = "0 0 0"/>
+    </visual>
+  </link>
+  <joint name = "panto_a3" type="revolute">
+    <parent link = "panto_left_link2"/>
+    <child link = "panto_tool0"/>
+    <origin xyz = "0.165 0 0" rpy="0 0 0"/>
+    <limit effort="1000.0" lower="-1.57" upper="1.57" velocity="0.5"/>
+    <axis xyz = "0 0 1"/>
+    <dynamics damping="0.2" friction="0.1" />
+  </joint>
   <!-- ==========  Right arm (as seen from behind) =========== -->
   <link name = "panto_right_motor">
-    <visual>
-      <geometry>
-        <cylinder length = "0.1" radius = "0.05"/>
-      </geometry>
-      <material name = "green"/>
-      <origin xyz = "0 0 0.05"/>
-    </visual>
+    <inertial>
+      <!-- izz = 69.9 g/cm², see https://www.farnell.com/datasheets/484832.pdf -->
+      <mass value="0.1"/>
+      <inertia ixx="0.1" ixy="0.0" ixz="0.0" iyy="0.1" iyz="0.0" izz="0.00000699"/>
+    </inertial>
   </link>
-  <joint name = "panto_right_joint" type="revolute">
+  <joint name = "panto_a5" type="revolute">
     <parent link = "panto_base"/>
     <child link = "panto_right_motor"/>
-    <origin xyz = "0.041 0 0" rpy="0 0 0"/>
+    <origin xyz = "0.085 0 0" rpy="0 0 0"/>
     <limit effort="1000.0" lower="-1.57" upper="1.57" velocity="0.5"/>
     <axis xyz = "0 0 1"/>
@@ -47,7 +128,7 @@
     <visual>
       <geometry>
-        <box size = "0.1 0.03 0.03"/>
+        <mesh filename="package://pantograph_description/meshes/mesh_link_left_1.stl" scale="0.001 0.001 0.001"/>
       </geometry>
-      <material name = "blue"/>
+      <material name = "green"/>
       <origin xyz = "0 0 0" rpy = "0 0 0"/>
     </visual>
@@ -58,42 +139,21 @@
     <origin xyz = "0 0 0"/>
   </joint>
-  <!--
   <link name = "panto_right_link2">
     <visual>
       <geometry>
-        <box size = "0.165 0.03 0.03"/>
+        <mesh filename="package://pantograph_description/meshes/mesh_link_right_2.stl" scale="0.001 0.001 0.001"/>
       </geometry>
-      <material name = "blue"/>
-      <origin xyz = "0.0825 0 0" rpy = "0 0 0" />
+      <material name = "green"/>
+      <origin xyz = "0 0 0" rpy = "0 0 0"/>
     </visual>
   </link>
-  <joint name = "panto_right_joint2" type="revolute">
+  <joint name = "panto_a4" type="revolute">
     <parent link = "panto_right_link1"/>
     <child link = "panto_right_link2"/>
-    <origin xyz = "0.3 0 0.13"/>
+    <origin xyz = "0.1 0 0" rpy="0 0 0"/>
     <limit effort="1000.0" lower="-1.57" upper="1.57" velocity="0.5"/>
     <axis xyz = "0 0 1"/>
     <dynamics damping="0.2" friction="0.1" />
   </joint>
-  -->
-  <!-- ==========  Left arm (as seen from behind) =========== -->
-  <link name = "panto_left_motor">
-    <visual>
-      <geometry>
-        <cylinder length = "0.1" radius = "0.05"/>
-      </geometry>
-      <material name = "green"/>
-      <origin xyz = "0 0 0.05"/>
-    </visual>
-  </link>
-  <joint name = "panto_left_joint" type="revolute">
-    <parent link = "panto_base"/>
-    <child link = "panto_left_motor"/>
-    <origin xyz = "-0.041 0 0" rpy="0 0 0"/>
-    <limit effort="1000.0" lower="-1.57" upper="1.57" velocity="0.5"/>
-    <axis xyz = "0 0 1"/>
-    <dynamics damping="0.2" friction="0.1" />
-  </joint>
-  <!-- ==========  Tool link (orange sphere) =========== -->
   </xacro:macro>
 </robot>

Commit message: add needle to description pkg

File: pantograph_description/ros2_control/pantograph.r2c_hardware.xacro (robot description, xacro)
@@ -125,4 +125,21 @@
           </state_interface>
       </joint>
+<!--Test of universal joint at end efector-->
+      <joint name="tool_pitch_joint">
+          <command_interface name="position"/>
+          <state_interface name="position">
+            <param name="initial_value">${0}</param>
+            <param name="min">-3</param>
+            <param name="max">3</param>
+          </state_interface>
+      </joint>
+    <joint name="tool_roll_joint">
+        <command_interface name="position"/>
+        <state_interface name="position">
+          <param name="initial_value">${0}</param>
+          <param name="min">-3</param>
+          <param name="max">3</param>
+        </state_interface>
+    </joint>
     </ros2_control>
   </xacro:macro>

File: pantograph_description/urdf/pantograph.urdf.xacro (robot description, xacro)
@@ -156,4 +156,31 @@
     <dynamics damping="0.2" friction="0.1" />
   </joint>
+  <!-- ==========  Test universal joint at end effector =========== -->
+  <!-- tool pitch angle-->
+  <link name="tool_pitch_link"/>
+  <joint name="tool_pitch_joint" type="revolute">
+    <parent link= "panto_tool0"/>
+    <child link= "tool_pitch_link"/>
+    <origin xyz = "0 0 0" rpy="0 0 0"/>
+    <limit effort="1000.0" lower="-3" upper="3" velocity="0.5"/>
+    <axis xyz="0 1 0"/>
+  </joint>
+   <!-- tool roll angle-->
+   <link name = "tool_roll_link">
+     <visual>
+       <geometry>
+         <cylinder length = "0.2" radius = "0.0025"/>
+       </geometry>
+       <material name = "white_alpha"/>
+       <origin xyz = "0 0 0.1" rpy = "0 0 0"/>
+     </visual>
+   </link>
+   <joint name="tool_roll_joint" type="revolute">
+      <origin rpy="0 0 0" xyz="0 0 0"/>
+      <parent link="tool_pitch_link"/>
+      <child link="tool_roll_link"/>
+      <limit effort="1000.0" lower="-3" upper="3" velocity="0.5"/>
+      <axis xyz="1 0 0"/>
+   </joint>
   </xacro:macro>
 </robot>

Commit message: added tool_orientation_controller for testing of universal joint at end effector

File: pantograph_description/ros2_control/pantograph.r2c_hardware.xacro (robot description, xacro)
@@ -125,21 +125,21 @@
           </state_interface>
       </joint>
-<!--Test of universal joint at end efector-->
+      <!--Test of universal joint at end efector-->
       <joint name="tool_pitch_joint">
           <command_interface name="position"/>
-          <state_interface name="position">
+            <state_interface name="position">
+              <param name="initial_value">${0}</param>
+              <param name="min">-1.57</param>
+              <param name="max">1.57</param>
+            </state_interface>
+      </joint>
+      <joint name="tool_roll_joint">
+          <command_interface name="position"/>
+            <state_interface name="position">
             <param name="initial_value">${0}</param>
-            <param name="min">-3</param>
-            <param name="max">3</param>
+            <param name="min">-1.57</param>
+            <param name="max">1.57</param>
           </state_interface>
       </joint>
-    <joint name="tool_roll_joint">
-        <command_interface name="position"/>
-        <state_interface name="position">
-          <param name="initial_value">${0}</param>
-          <param name="min">-3</param>
-          <param name="max">3</param>
-        </state_interface>
-    </joint>
     </ros2_control>
   </xacro:macro>

Commit message: changed joint names for clarification

File: pantograph_description/ros2_control/pantograph.r2c_hardware.xacro (robot description, xacro)
@@ -126,20 +126,37 @@
       </joint>
       <!--Test of universal joint at end efector-->
-      <joint name="tool_pitch_joint">
+      <joint name="tool_theta_joint">
           <command_interface name="position"/>
             <state_interface name="position">
               <param name="initial_value">${0}</param>
-              <param name="min">-1.57</param>
-              <param name="max">1.57</param>
+              <param name="min">-3</param>
+              <param name="max">3</param>
             </state_interface>
       </joint>
-      <joint name="tool_roll_joint">
+      <joint name="tool_phi_joint">
           <command_interface name="position"/>
             <state_interface name="position">
-            <param name="initial_value">${0}</param>
-            <param name="min">-1.57</param>
-            <param name="max">1.57</param>
+             <param name="initial_value">${0}</param>
+             <param name="min">-3</param>
+             <param name="max">3</param>
+            </state_interface>
+      </joint>
+      <!--Test of position controller for model verification-->
+      <!-- <joint name="panto_a1">
+          <command_interface name="position"/>
+            <state_interface name="position">
+             <param name="initial_value">${0}</param>
+             <param name="min">-1.57</param>
+             <param name="max">1.57</param>
+            </state_interface>
+      </joint>
+      <joint name="panto_a5">
+        <command_interface name="position"/>
+          <state_interface name="position">
+           <param name="initial_value">${0}</param>
+           <param name="min">-1.57</param>
+           <param name="max">1.57</param>
           </state_interface>
-      </joint>
+      </joint> -->
     </ros2_control>
   </xacro:macro>

File: pantograph_description/urdf/pantograph.urdf.xacro (robot description, xacro)
@@ -158,29 +158,29 @@
   <!-- ==========  Test universal joint at end effector =========== -->
   <!-- tool pitch angle-->
-  <link name="tool_pitch_link"/>
-  <joint name="tool_pitch_joint" type="revolute">
+  <link name="tool_theta_link"/>
+  <joint name="tool_theta_joint" type="revolute">
     <parent link= "panto_tool0"/>
-    <child link= "tool_pitch_link"/>
+    <child link= "tool_theta_link"/>
     <origin xyz = "0 0 0" rpy="0 0 0"/>
+    <limit effort="1000.0" lower="-3" upper="3" velocity="0.5"/>
+    <axis xyz="0 0 1"/>
+  </joint>
+  <!-- tool roll angle-->
+  <link name = "tool_phi_link">
+    <visual>
+      <geometry>
+        <cylinder length = "0.2" radius = "0.0025"/>
+      </geometry>
+      <material name = "white_alpha"/>
+      <origin xyz = "0 0 0.1" rpy = "0 0 0"/>
+    </visual>
+  </link>
+  <joint name="tool_phi_joint" type="revolute">
+    <origin rpy="0 0 0" xyz="0 0 0"/>
+    <parent link="tool_theta_link"/>
+    <child link="tool_phi_link"/>
     <limit effort="1000.0" lower="-3" upper="3" velocity="0.5"/>
     <axis xyz="0 1 0"/>
   </joint>
-   <!-- tool roll angle-->
-   <link name = "tool_roll_link">
-     <visual>
-       <geometry>
-         <cylinder length = "0.2" radius = "0.0025"/>
-       </geometry>
-       <material name = "white_alpha"/>
-       <origin xyz = "0 0 0.1" rpy = "0 0 0"/>
-     </visual>
-   </link>
-   <joint name="tool_roll_joint" type="revolute">
-      <origin rpy="0 0 0" xyz="0 0 0"/>
-      <parent link="tool_pitch_link"/>
-      <child link="tool_roll_link"/>
-      <limit effort="1000.0" lower="-3" upper="3" velocity="0.5"/>
-      <axis xyz="1 0 0"/>
-   </joint>
   </xacro:macro>
 </robot>

Commit message: added prismatic joint for modelling of needle insertion

File: pantograph_description/ros2_control/pantograph.r2c_hardware.xacro (robot description, xacro)
@@ -142,21 +142,13 @@
             </state_interface>
       </joint>
-      <!--Test of position controller for model verification-->
-      <!-- <joint name="panto_a1">
-          <command_interface name="position"/>
-            <state_interface name="position">
-             <param name="initial_value">${0}</param>
-             <param name="min">-1.57</param>
-             <param name="max">1.57</param>
-            </state_interface>
-      </joint>
-      <joint name="panto_a5">
+      <!--Test of needle interaction point-->
+      <joint name="needle_interaction_joint">
         <command_interface name="position"/>
           <state_interface name="position">
            <param name="initial_value">${0}</param>
-           <param name="min">-1.57</param>
-           <param name="max">1.57</param>
+           <param name="min">-0.5</param>
+           <param name="max">0.5</param>
           </state_interface>
-      </joint> -->
+      </joint>
     </ros2_control>
   </xacro:macro>

File: pantograph_description/urdf/pantograph.urdf.xacro (robot description, xacro)
@@ -181,4 +181,13 @@
     <axis xyz="0 1 0"/>
   </joint>
+  <!-- ==========  Test needle insertion DoF =========== -->
+  <link name = "needle_interaction_link"/>
+  <joint name="needle_interaction_joint" type="prismatic">
+    <parent link= "tool_phi_link"/>
+    <child link= "needle_interaction_link"/>
+    <origin xyz = "0 0 0.1" rpy="0 0 0"/>
+    <limit effort="1000.0" lower="0.5" upper="-0.5" velocity="0.5"/>
+    <axis xyz="0 0 1"/>
+  </joint>
   </xacro:macro>
 </robot>
